File: projects/gartenbewaesserung/kicad/pumpensteuerung/tht/relaismodule.kicad_sch (KiCad schematic)
At the start: 5 parts, among them J1 Screw_Terminal_01x03, K2 SANYOU_SRD_Form_C, Q1 S8050

Commit message: [gartenbewaesserung(pcb)] replace fake footprints with real one
Parts:
- J1: footprint TerminalBlock:TerminalBlock_Altech_AK300-3_P5.00mm -> PhoenixContact:MKDSN 1,5_3-5,08
Changed lines of the file:
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@@
 			)
 		)
-		(property "Footprint" "TerminalBlock:TerminalBlock_Altech_AK300-3_P5.00mm"
+		(property "Footprint" "PhoenixContact:MKDSN 1,5_3-5,08"
 			(at 82.55 41.91 0)
 			(effects
